File: SenDes_Project.kicad_sch (KiCad schematic)
At the start: 2 parts, among them U1 ESP32-S3-WROOM-1, U2 TCAN332

Commit message: Add files via upload
Parts:
- added J1: Conn_01x02_Pin, symbol Connector:Conn_01x02_Pin
- added U3, U4: MP1584 Buck Module - 5V, symbol SenDes_custom_symbols:Buck_Converter_Module
- added U5: MP1584 Buck Module - 3.3V, symbol SenDes_custom_symbols:Buck_Converter_Module
Other:
- moved on the sheet: U1

Commit message: Add files via upload
Parts:
- added U6, U7: TPS4HC120-Q1, symbol SenDes_custom_symbols:TPS4HC120-Q1
- added U8: MP1584 Buck Module - 3.3V, symbol SenDes_custom_symbols:Buck_Converter_Module

Commit message: Add files via upload
Parts:
- removed U1: ESP32-S3-WROOM-1, RF_Module:ESP32-S3-WROOM-1, symbol RF_Module:ESP32-S3-WROOM-1
- removed U2: TCAN332, symbol Interface_CAN_LIN:TCAN332
- removed U3, U4: MP1584 Buck Module - 5V, symbol SenDes_custom_symbols:Buck_Converter_Module
- removed U5, U8: MP1584 Buck Module - 3.3V, symbol SenDes_custom_symbols:Buck_Converter_Module
- removed U6, U7: TPS4HC120-Q1, symbol SenDes_custom_symbols:TPS4HC120-Q1
Other:
- added sheet CAN (CNH_Tester_can.kicad_sch)
- added sheet MCU (untitled.kicad_sch)
- added sheet Power Distribution (CNH_Tester_power_distribution.kicad_sch)
